Commit message: Progress so far

File: experiments/robots/crawler/assets/crawler.urdf (robot description, URDF)
Before this commit: robot URDF, 13 links, 12 joints
Links:
- added link leg_1_foot, mass 0.0014224078597118738; collision mesh filename=meshes/foot.stl scale=0.001 0.001 0.001; visual mesh filename=meshes/foot.stl scale=0.001 0.001 0.001
- added link leg_2_foot, mass 0.0014224078597118738; collision mesh filename=meshes/foot.stl scale=0.001 0.001 0.001; visual mesh filename=meshes/foot.stl scale=0.001 0.001 0.001
- added link leg_3_foot, mass 0.0014224078597118738; collision mesh filename=meshes/foot.stl scale=0.001 0.001 0.001; visual mesh filename=meshes/foot.stl scale=0.001 0.001 0.001
- added link leg_4_foot, mass 0.0014224078597118738; collision mesh filename=meshes/foot.stl scale=0.001 0.001 0.001; visual mesh filename=meshes/foot.stl scale=0.001 0.001 0.001
- link leg_1_tibia: mass 0.01570347323772935 -> 0.014281065378017476
- link leg_2_tibia: mass 0.01570347323772935 -> 0.014281065378017476
- link leg_3_tibia: mass 0.01570347323772935 -> 0.014281065378017476
- link leg_4_tibia: mass 0.01570347323772935 -> 0.014281065378017476
Joints:
- removed joint leg_1_coxa
- removed joint leg_1_femur
- removed joint leg_1_tibia
- removed joint leg_2_coxa
- removed joint leg_2_femur
- removed joint leg_2_tibia
- removed joint leg_3_coxa
- removed joint leg_3_femur
- removed joint leg_3_tibia
- removed joint leg_4_coxa
- removed joint leg_4_femur
- removed joint leg_4_tibia
- added joint base_leg_1_coxa: type continuous, parent base, child leg_1_coxa, origin xyz=-0.02249999588670991 -0.02250000396793932 -4.682672214428862e-09 rpy=3.141592653589793 -0.0 -1.5707963267948966, axis 0.0 0.0 1.0
- added joint base_leg_2_coxa: type continuous, parent base, child leg_2_coxa, origin xyz=-0.02249999588670991 0.022499996032060682 -4.682672214428862e-09 rpy=3.141592653589793 -0.0 -1.5707963267948966, axis 0.0 0.0 1.0
- added joint base_leg_3_coxa: type continuous, parent base, child leg_3_coxa, origin xyz=0.022500004113290083 0.022499996032060682 -4.682672214428862e-09 rpy=3.141592653589793 -0.0 -1.5707963267948966, axis 0.0 0.0 1.0
- added joint base_leg_4_coxa: type continuous, parent base, child leg_4_coxa, origin xyz=0.022500004113290083 -0.02250000396793932 -4.682672214428862e-09 rpy=3.141592653589793 -0.0 -1.5707963267948966, axis 0.0 0.0 1.0
- added joint leg_1_coxa_leg_1_femur: type continuous, parent leg_1_coxa, child leg_1_femur, origin xyz=0.012020810000000002 0.007778179999999999 -0.006999999999999999 rpy=3.141592653589793 5.416677968589073e-35 0.0, axis 0.707107 0.707107 3.830170908335114e-35
- added joint leg_1_femur_leg_1_tibia: type continuous, parent leg_1_femur, child leg_1_tibia, origin xyz=0.02828427 -0.028284270000000004 0.0 rpy=1.5407439555097883e-33 9.013165799496008e-34 -2.4651903288156613e-32, axis -0.7071070000000002 -0.707107 -4.84832862692823e-33
- added joint leg_1_tibia_leg_1_foot: type fixed, parent leg_1_tibia, child leg_1_foot, origin xyz=0.021465179999999997 -0.02570782 -2.220446049250313e-18 rpy=1.5707963267948966 -8.471498002637101e-34 2.465190328815662e-32
- added joint leg_2_coxa_leg_2_femur: type continuous, parent leg_2_coxa, child leg_2_femur, origin xyz=-0.008340729999999992 0.01258337 -0.006999999999999999 rpy=3.141592653589793 -5.416677968589073e-35 0.0, axis 0.707107 -0.707107 -3.830170908335114e-35
- added joint leg_2_femur_leg_2_tibia: type continuous, parent leg_2_femur, child leg_2_tibia, origin xyz=-0.028284270000000014 -0.028284270000000004 0.0 rpy=-6.162975822039155e-33 1.5152067497230174e-33 4.930380657631324e-32, axis -0.707107 0.707107 -1.631123776889653e-32
- added joint leg_2_tibia_leg_2_foot: type fixed, parent leg_2_tibia, child leg_2_foot, origin xyz=-0.025707819999999996 -0.02146518 0.0 rpy=1.5707963267948966 -1.569373529408908e-33 -4.930380657631324e-32
- added joint leg_3_coxa_leg_3_femur: type continuous, parent leg_3_coxa, child leg_3_femur, origin xyz=-0.01258337 -0.008340720000000008 -0.006999999999999999 rpy=3.141592653589793 2.116374158186469e-30 1.9721522630525295e-31, axis -0.707107 -0.707107 -1.6254898759704362e-30
- added joint leg_3_femur_leg_3_tibia: type continuous, parent leg_3_femur, child leg_3_tibia, origin xyz=-0.028284269999999997 0.028284269999999997 0.0 rpy=-4.173812085533337e-61 -2.200041170737885e-31 3.944304526105059e-31, axis 0.707107 0.707107 1.876117590738102e-30
- added joint leg_3_tibia_leg_3_foot: type fixed, parent leg_3_tibia, child leg_3_foot, origin xyz=-0.021465180000000004 0.025707820000000013 0.0 rpy=1.5707963267948966 2.3363782752602575e-30 -5.9164567891575885e-31
- added joint leg_4_coxa_leg_4_femur: type continuous, parent leg_4_coxa, child leg_4_femur, origin xyz=0.007778170000000002 -0.012020810000000015 -0.006999999999999999 rpy=3.141592653589793 -2.205677087359668e-33 1.232595164407831e-32, axis -0.707107 0.7071069999999999 -3.241300140912161e-33
- added joint leg_4_femur_leg_4_tibia: type continuous, parent leg_4_femur, child leg_4_tibia, origin xyz=0.02828427 0.028284270000000014 -2.220446049250313e-18 rpy=6.162975822039157e-33 7.672534297059725e-33 1.2325951644078312e-32, axis 0.707107 -0.7071070000000002 -1.0367299274946627e-32
- added joint leg_4_tibia_leg_4_foot: type fixed, parent leg_4_tibia, child leg_4_foot, origin xyz=0.02570782 0.021465180000000004 0.0 rpy=1.5707963267948966 -8.263406457993844e-34 0.0
